File: MSP430G2553-with-dac/_autosave-MSP430G2553-with-dac.kicad_pcb (KiCad board)
At the start: 2 copper layers, 55.9 x 43.2 mm, 19 parts, among them IC1 MX25L4006E, P1 DEBUG, P2 OUT, P3 PHOTODIODE, Q1 2N3906, SW1 PEL12T, U1 MSP430G2553IN20, U2 MCP4922-E/P

Commit message: 430/DAC board laid out. Probably badly
Routing:
- net /BUTTON: track 0.65 -> 27.7 mm, vias 0 -> 1
- net GND: track 0.00 -> 9.11 mm, vias 0 -> 5
- net /RXD: track 42.4 -> 42.9 mm, vias 0 -> 2
