File: MSP430G2553-with-dac/MSP430G2553-with-dac.kicad_pcb (KiCad board)
At the start: 2 copper layers, 55.9 x 43.2 mm, 19 parts, among them IC1 MX25L4006E, P1 DEBUG, P2 OUT, P3 PHOTODIODE, Q1 2N3906, SW1 PEL12T, U1 MSP430G2553IN20, U2 MCP4922-E/P

Commit message: Ready for manufacture.
Parts:
- added ?: , Mounting_Holes:MountingHole_2-5mm, F.Cu at (130.8, 110.5)
- added ?: , Mounting_Holes:MountingHole_2-5mm, F.Cu at (130.8, 146.1)
- added ?: , Mounting_Holes:MountingHole_2-5mm, F.Cu at (179.1, 146.1)
- added ?: , Mounting_Holes:MountingHole_2-5mm, F.Cu at (179.1, 110.5)
- moved P3 1.91 mm to (176.5, 116.2)
Routing:
- net /BUTTON: track 0.65 -> 27.7 mm, vias 0 -> 1
- net /TXD: track 48.4 -> 58.8 mm
- net GND: track 0.00 -> 9.11 mm, vias 0 -> 5
- net Net-(P3-Pad1): track 15.6 -> 14.0 mm
- net /RXD: track 42.4 -> 41.1 mm, vias 0 -> 2
- net /RST#: track 41.1 -> 42.4 mm
- net /SDO: track 50.9 -> 50.0 mm
- net /PH_IN: track 34.3 -> 33.5 mm
- net /TEST: track 32.1 -> 31.3 mm
Other:
- board text added: "+"
- board text added: "-"
- board text added: "MPS430G2553 with Flash and DAC"

Commit message: Cosmetic changes + start firmware.
Changed lines of the file:
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@@
     (pad 6 thru_hole oval (at 2.5 7.5 90) (size 1.8 2.1) (drill 1.1) (layers *.Cu *.Mask F.SilkS)
       (net 23 /Q_B))
-    (pad "" np_thru_hole rect (at 5.6 0 180) (size 2.4 2) (drill oval 2.1 1) (layers *.Cu *.Mask F.SilkS))
-    (pad "" np_thru_hole rect (at -5.6 0 180) (size 2.4 2) (drill oval 2.1 1) (layers *.Cu *.Mask F.SilkS))
+    (pad "" np_thru_hole circle (at 5.6 0 180) (size 2.8 2.8) (drill 2.1) (layers *.Cu *.Mask F.SilkS))
+    (pad "" np_thru_hole circle (at -5.6 0 180) (size 2.8 2.8) (drill 2.1) (layers *.Cu *.Mask F.SilkS))
   )
   (gr_text - (at 180.975 134.62) (layer F.SilkS)
